File: CM5IO.kicad_pcb (KiCad board)
At the start: 4 copper layers, 160 x 90 mm, 79 parts, among them J10 690-019-298-412, J11 USB_C_Receptacle_USB2.0, J12 USB3_A, J14 JST_SHBM04B-SRSS-TB, J16 Conn_01x22_Female, J2 Conn_02x07_Odd_Even, J22 690-019-298-412, J3 Conn_01x03, J4 Bus_M.2_Socket_M, J5 Conn_01x22_Female, J6 THD-02-R, J7 Micro_SD_Card_Det, J8 THD-20-R, J9 THD-02-R, SW1 Right angle Tact button, U1 TPD4EUSB30, U12 RT9742SNGV, U18 RT9742GGJ5, U2 TPD4EUSB30, U3 MagJack-A70-112-331N126, U6 AP22653W6, U7 ASEK-32.768KHZ-L-R-T, U8 AP3441SHE-7B

Commit message: whatever
Parts:
- removed BT1: Battery_Cell, CM5IO:BatteryHolder_Keystone_3034_1x20mm
- removed C15, C16, C17: 10u, Capacitor_SMD:C_0805_2012Metric
- removed C19: 100n, Capacitor_SMD:C_0402_1005Metric
- removed D1: LED Red, LED_SMD:LED_0603_1608Metric
- removed D2: LED Green, LED_SMD:LED_0603_1608Metric
- removed H1, H2, H3, H4, H5, H6, H7, H8: MountingHole, CM5IO:MountingHole_2.7mm_M2.5_DIN965
- removed J10: 690-019-298-412, CM5IO:EDAC 690-019-298-412
- removed J14: JST_SHBM04B-SRSS-TB, Connector_JST:JST_SH_BM04B-SRSS-TB_1x04-1MP_P1.00mm_Vertical
- removed J3: Conn_01x03, Connector_PinHeader_2.54mm:PinHeader_1x03_P2.54mm_Vertical
- removed J6: THD-02-R, Connector_PinHeader_2.54mm:PinHeader_2x02_P2.54mm_Vertical
- removed L1: 2.2uH, CM5IO:L_Bourns_SRP5030CC
- removed R1, R10, R17: 1k, Resistor_SMD:R_0402_1005Metric
- removed R11, R13, R15: 10K 1%, Resistor_SMD:R_0402_1005Metric
- removed R14: 100K 1%, Resistor_SMD:R_0402_1005Metric
- removed R16: 2.2K 1%, Resistor_SMD:R_0402_1005Metric
- removed REF**: KiCad-Logo2_5mm_SilkScreen, Symbol:KiCad-Logo2_5mm_SilkScreen
- removed SW1: Right angle Tact button, Button_Switch_THT:SW_Tactile_SPST_Angled_PTS645Vx58-2LFS
- removed U18: RT9742GGJ5, Package_TO_SOT_SMD:SOT-23-5
- removed U7: ASEK-32.768KHZ-L-R-T, Crystal:Crystal_SMD_3225-4Pin_3.2x2.5mm
- removed U8: AP3441SHE-7B, Package_DFN_QFN:DFN-8-1EP_2x2mm_P0.5mm_EP1.05x1.75mm
- added CP1: 10uF, Capacitor_Tantalum_SMD:CP_EIA-3528-21_Kemet-B_HandSolder, F.Cu at (161.3, 136.2)
- added CP2: 22uF, Capacitor_Tantalum_SMD:CP_EIA-3528-21_Kemet-B_HandSolder, F.Cu at (168.2, 128.3)
- added CP3: 22uF, Capacitor_Tantalum_SMD:CP_EIA-3528-21_Kemet-B_HandSolder, F.Cu at (168.2, 131.9)
- added CP4: 100nF, Capacitor_SMD:C_0805_2012Metric_Pad1.18x1.45mm_HandSolder, F.Cu at (165.1, 134.9)
- added CP5: 2.7nF, Capacitor_SMD:C_0805_2012Metric_Pad1.18x1.45mm_HandSolder, F.Cu at (173.2, 137.2)
- added CP6: 33pF, Capacitor_SMD:C_0805_2012Metric_Pad1.18x1.45mm_HandSolder, F.Cu at (176.3, 138.2)
- added CP7: 10nF, Capacitor_SMD:C_0805_2012Metric_Pad1.18x1.45mm_HandSolder, F.Cu at (163.3, 142.3)
- added CP8: OPEN, Capacitor_SMD:C_0805_2012Metric_Pad1.18x1.45mm_HandSolder, F.Cu at (173.2, 141.3)
- added D4: MBR1020VL, Diode_SMD:D_SOD-123F, F.Cu at (248.7, 125.0)
- added H10: GND_SOLDERPOINT, Connector_Wire:SolderWirePad_1x01_SMD_5x10mm, F.Cu at (152.4, 136.3)
- added H9: VIN_SOLDERPOINT, Connector_Wire:SolderWirePad_1x01_SMD_5x10mm, F.Cu at (152.4, 141.9)
- added J1: POWER TERMINAL, TerminalBlock:TerminalBlock_bornier-2_P5.08mm, F.Cu at (150.5, 141.7)
- added JP1: ADDR1, Jumper:SolderJumper-3_P2.0mm_Open_TrianglePad1.0x1.5mm, F.Cu at (243.3, 142.4)
- added JP2: ADDR2, Jumper:SolderJumper-3_P2.0mm_Open_TrianglePad1.0x1.5mm, F.Cu at (243.3, 145.2)
- added JP3: ADDR4, Jumper:SolderJumper-3_P2.0mm_Open_TrianglePad1.0x1.5mm, F.Cu at (243.3, 148.0)
- added JP4: ADDR8, Jumper:SolderJumper-3_P2.0mm_Open_TrianglePad1.0x1.5mm, F.Cu at (243.3, 150.8)
- added JP5: ADDR16, Jumper:SolderJumper-3_P2.0mm_Open_TrianglePad1.0x1.5mm, F.Cu at (243.3, 153.6)
- added JP8: BT_WIFI_DISABLE, Jumper:SolderJumper-3_P2.0mm_Open_TrianglePad1.0x1.5mm, F.Cu at (199.6, 84.3)
- added LP1: 3.6uH, Inductor_SMD:L_Bourns-SRN8040_8x8.15mm, F.Cu at (175.3, 131.6)
- added RP1: 115K, Resistor_SMD:R_0805_2012Metric_Pad1.20x1.40mm_HandSolder, F.Cu at (173.2, 143.3)
- added RP2: 22.1K, Resistor_SMD:R_0805_2012Metric_Pad1.20x1.40mm_HandSolder, F.Cu at (169.4, 143.3)
- added RP3: 15.8K, Resistor_SMD:R_0805_2012Metric_Pad1.20x1.40mm_HandSolder, F.Cu at (173.2, 139.3)
- added SW2: SW_RESET, Button_Switch_SMD:SW_Push_1P1T_NO_CK_KMR2, F.Cu at (261.6, 132.6)
- added SW3: SW_BOOT, Button_Switch_SMD:SW_Push_1P1T_NO_CK_KMR2, F.Cu at (255.0, 132.6)
- added SW4: FORCE_EN, Button_Switch_SMD:SW_Push_1P1T_NO_CK_KMR2, F.Cu at (159.5, 142.9)
- added TP6: TestPoint, TestPoint:TestPoint_Pad_2.0x2.0mm, F.Cu at (276.6, 104.3)
- added UP1: AP64501SP-13, CM5IO:SOP_AP64501SP-13_DIO, F.Cu at (167.5, 138.6)
- C1: value 100n -> 4.7uF 25v; footprint Capacitor_SMD:C_0402_1005Metric -> Capacitor_Tantalum_SMD:CP_EIA-3528-21_Kemet-B_HandSolder
- C10: value 100n -> 4.7uF 6.3v; footprint Capacitor_SMD:C_0402_1005Metric -> Capacitor_Tantalum_SMD:CP_EIA-3216-18_Kemet-A_HandSolder
- C11: value 4.7nF -> 470nF; footprint Capacitor_SMD:C_0402_1005Metric -> Capacitor_SMD:C_0805_2012Metric_Pad1.18x1.45mm_HandSolder
- C12, C2, C7, C8, J7, R12, U12, U6: moved to B.Cu
- C14: value 10u -> 470nF; footprint Capacitor_SMD:C_0805_2012Metric -> Capacitor_SMD:C_0805_2012Metric_Pad1.18x1.45mm_HandSolder
- C4: value 10u -> 4.7uF 6.3v; footprint Capacitor_SMD:C_0805_2012Metric -> Capacitor_Tantalum_SMD:CP_EIA-3216-18_Kemet-A_HandSolder
- C6: value 10u -> 4.7uF 25v; footprint Capacitor_SMD:C_0805_2012Metric -> Capacitor_Tantalum_SMD:CP_EIA-3528-21_Kemet-B_HandSolder
- D3: value LED Green -> MBR1020VL; footprint LED_SMD:LED_0603_1608Metric -> Diode_SMD:D_SOD-123F
- J12: footprint CM5IO:MTCONN_UBAF30-D2011 -> Connector_USB:USB3_A_Molex_48393-001
- J2: value Conn_02x07_Odd_Even -> Conn_02x06_Odd_Even; footprint Connector_PinHeader_2.54mm:PinHeader_2x07_P2.54mm_Vertical -> Connector_PinHeader_1.27mm:PinHeader_2x06_P1.27mm_Vertical
- J22: value 690-019-298-412 -> 46765-1301; footprint CM5IO:EDAC 690-019-298-412 -> CM5IO:CONN_467651301_MOL
- J4: value Bus_M.2_Socket_M -> ESP_UART; footprint CM5IO:M.2 M Key socket -> Connector_PinSocket_2.54mm:PinSocket_1x04_P2.54mm_Vertical
- J9: value THD-02-R -> USB_C_Receptacle_USB2.0; footprint Connector_PinHeader_2.54mm:PinHeader_2x02_P2.54mm_Vertical -> Connector_USB:USB_C_Receptacle_GCT_USB4105-xx-A_16P_TopMnt_Horizontal
- R2: value 470R -> 1K; footprint Resistor_SMD:R_0402_1005Metric -> Resistor_SMD:R_0805_2012Metric_Pad1.20x1.40mm_HandSolder
- R3: value 470R -> 2.2K 1%; footprint Resistor_SMD:R_0402_1005Metric -> Resistor_SMD:R_0805_2012Metric_Pad1.20x1.40mm_HandSolder
- R4: value nf -> 1K
- R5: value 0R -> 1K
- TP1, TP2, TP3, TP4, TP5: moved to F.Cu
- U1: value TPD4EUSB30 -> AP7361C-33E; footprint Package_SON:USON-10_2.5x1.0mm_P0.5mm -> Package_TO_SOT_SMD:SOT-223-3_TabPin2
- U2: value TPD4EUSB30 -> ESP32-S3-WROOM-1; footprint Package_SON:USON-10_2.5x1.0mm_P0.5mm -> RF_Module:ESP32-S3-WROOM-1; moved to B.Cu
- U3: value MagJack-A70-112-331N126 -> AP7361C-33E; footprint CM5IO:TRJG0926HENL -> Package_TO_SOT_SMD:SOT-223-3_TabPin2
- moved TP5 167.1 mm to (276.6, 121.6)
- moved TP3 165.9 mm to (276.6, 113.0)
- moved J9 137.6 mm to (226.6, 43.4), turned to 0 degrees
- moved J8 114.8 mm to (201.2, 93.2), turned to 0 degrees
- moved R3 113.9 mm to (220.2, 41.3)
- moved U2 113.2 mm to (261.2, 155.9), turned to 0 degrees
- moved C1 110.4 mm to (258.6, 108.4), turned to 0 degrees
- moved U3 103.8 mm to (250.8, 115.9)
- moved U1 100.3 mm to (250.8, 107.6), turned to 0 degrees
- moved R4 86.4 mm to (264.6, 131.6), turned to 90 degrees
- moved TP1 86.0 mm to (276.6, 100.0)
- moved R2 79.7 mm to (242.3, 140.0), turned to 180 degrees
- moved R5 79.7 mm to (258.0, 131.6), turned to 90 degrees
- moved TP4 79.4 mm to (276.6, 117.3), turned to 0 degrees
- moved C12 78.2 mm to (155.4, 84.8)
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Connections:
- C1 pad 1: Net-(C1-Pad1) -> /LoRa/VIN
- C10 pad 1: /+5v -> /LoRa/+3.3v_LoRa
- C11 pad 1: /PCIe-M2/M2_3v3 -> GND
- C11 pad 2: /PCIe-M2/FB -> /LoRa/BOOT_MODE
- C14 pad 1: /PCIe-M2/M2_3v3 -> GND
- C14 pad 2: GND -> /LoRa/ENABLE
- C4 pad 1: /+5v -> /LoRa/+3.3v_ESP
- C6 pad 1: /+5v -> /LoRa/VIN
- D3 pad 1: Net-(D3-K) -> /LoRa/VIN
- D3 pad 2: /PCIe-M2/M2_3v3 -> /LoRa/+5v
- J2 pad 10: /CM5_GPIO ( Ethernet, GPIO, SDCARD)/USBOTG -> /CM5_GPIO ( Ethernet, GPIO, SDCARD)/PMIC_ENABLE
- J2 pad 12: /CM5_GPIO ( Ethernet, GPIO, SDCARD)/PMIC_ENABLE -> /CM5_GPIO ( Ethernet, GPIO, SDCARD)/PWR_BUT
- J2 pad 8: unconnected-(J2-Pin_8-Pad8) -> /CM5_GPIO ( Ethernet, GPIO, SDCARD)/USBOTG
- J22 pad 1: /CM5_HighSpeed/HDMI0_D2_P -> /CM5_HighSpeed/HDMI0_HOTPLUG
- J22 pad 10: /CM5_HighSpeed/HDMI0_CK_P -> GND
- J22 pad 11: GND -> /CM5_HighSpeed/HDMI0_D0_N
- J22 pad 12: /CM5_HighSpeed/HDMI0_CK_N -> /CM5_HighSpeed/HDMI0_CK_P
- J22 pad 13: /CM5_HighSpeed/HDMI0_CEC -> GND
- J22 pad 14: unconnected-(J22-UTILITY/HEAC+-Pad14) -> /CM5_HighSpeed/HDMI0_CK_N
- J22 pad 15: /CM5_HighSpeed/HDMI0_SCL -> /CM5_HighSpeed/HDMI0_CEC
- J22 pad 16: /CM5_HighSpeed/HDMI0_SDA -> GND
- J22 pad 17: GND -> /CM5_HighSpeed/HDMI0_SCL
- J22 pad 18: /CM5_HighSpeed/HDMI_5v -> /CM5_HighSpeed/HDMI0_SDA
- J22 pad 19: /CM5_HighSpeed/HDMI0_HOTPLUG -> /CM5_HighSpeed/HDMI_5v
- J22 pad 2: GND -> unconnected-(J22-UTILITY/HEAC+-Pad2)
- J22 pad 3: /CM5_HighSpeed/HDMI0_D2_N -> /CM5_HighSpeed/HDMI0_D2_P
- J22 pad 4: /CM5_HighSpeed/HDMI0_D1_P -> GND
- J22 pad 5: GND -> /CM5_HighSpeed/HDMI0_D2_N
- J22 pad 6: /CM5_HighSpeed/HDMI0_D1_N -> /CM5_HighSpeed/HDMI0_D1_P
- J22 pad 7: /CM5_HighSpeed/HDMI0_D0_P -> GND
- J22 pad 8: GND -> /CM5_HighSpeed/HDMI0_D1_N
- J22 pad 9: /CM5_HighSpeed/HDMI0_D0_N -> /CM5_HighSpeed/HDMI0_D0_P
- J4 pad 1: GND -> /LoRa/+3.3v_ESP
- J4 pad 2: /PCIe-M2/M2_3v3 -> Net-(J4-Pin_2)
- J4 pad 3: GND -> Net-(J4-Pin_3)
- J4 pad 4: /PCIe-M2/M2_3v3 -> GND
- J8 pad 27: /CM5_GPIO ( Ethernet, GPIO, SDCARD)/ID_SD -> unconnected-(J8-Pin_27-Pad27)
- J8 pad 28: /CM5_GPIO ( Ethernet, GPIO, SDCARD)/ID_SC -> unconnected-(J8-Pin_28-Pad28)
- Module1 pad 102: /CM5_HighSpeed/PCIE_nCLKREQ -> unconnected-(Module1B-PCIe_nCLKREQ-Pad102)
- Module1 pad 104: /CM5_HighSpeed/PCIE_nWAKE -> unconnected-(Module1B-PCIE_nWAKE-Pad104)
- Module1 pad 106: /CM5_HighSpeed/PCIE_PWR_EN -> unconnected-(Module1B-PCIE_PWR_EN-Pad106)
- Module1 pad 109: /CM5_HighSpeed/PCIE_nRST -> unconnected-(Module1B-PCIe_nRST-Pad109)
- Module1 pad 110: /CM5_HighSpeed/PCIE_CLK_P -> unconnected-(Module1B-PCIe_CLK_P-Pad110)
- Module1 pad 112: /CM5_HighSpeed/PCIE_CLK_N -> unconnected-(Module1B-PCIe_CLK_N-Pad112)
- Module1 pad 116: /CM5_HighSpeed/PCIE_RX_P -> unconnected-(Module1B-PCIe_RX_P-Pad116)
- Module1 pad 118: /CM5_HighSpeed/PCIE_RX_N -> unconnected-(Module1B-PCIe_RX_N-Pad118)
- Module1 pad 122: /CM5_HighSpeed/PCIE_TX_P -> unconnected-(Module1B-PCIe_TX_P-Pad122)
- Module1 pad 124: /CM5_HighSpeed/PCIE_TX_N -> unconnected-(Module1B-PCIe_TX_N-Pad124)
- Module1 pad 143: /CM5_HighSpeed/HDMI1_HOTPLUG -> unconnected-(Module1B-HDMI1_HOTPLUG-Pad143)
- Module1 pad 145: /CM5_HighSpeed/HDMI1_SDA -> unconnected-(Module1B-HDMI1_SDA-Pad145)
- Module1 pad 146: /CM5_HighSpeed/HDMI1_D2_P -> unconnected-(Module1B-HDMI1_TX2_P-Pad146)
- Module1 pad 147: /CM5_HighSpeed/HDMI1_SCL -> unconnected-(Module1B-HDMI1_SCL-Pad147)
- Module1 pad 148: /CM5_HighSpeed/HDMI1_D2_N -> unconnected-(Module1B-HDMI1_TX2_N-Pad148)
- Module1 pad 149: /CM5_HighSpeed/HDMI1_CEC -> unconnected-(Module1B-HDMI1_CEC-Pad149)
- Module1 pad 15: /CM5_GPIO ( Ethernet, GPIO, SDCARD)/ETH_LEDY -> unconnected-(Module1A-Ethernet_nLED3(3.3v)-Pad15)
- Module1 pad 152: /CM5_HighSpeed/HDMI1_D1_P -> unconnected-(Module1B-HDMI1_TX1_P-Pad152)
- Module1 pad 154: /CM5_HighSpeed/HDMI1_D1_N -> unconnected-(Module1B-HDMI1_TX1_N-Pad154)
- Module1 pad 157: /CM5_HighSpeed/USB3-1-RX_N -> unconnected-(Module1B-USB3-1-RX_N-Pad157)
- Module1 pad 158: /CM5_HighSpeed/HDMI1_D0_P -> unconnected-(Module1B-HDMI1_TX0_P-Pad158)
- Module1 pad 159: /CM5_HighSpeed/USB3-1-RX_P -> unconnected-(Module1B-USB3-1-RX_P-Pad159)
- Module1 pad 160: /CM5_HighSpeed/HDMI1_D0_N -> unconnected-(Module1B-HDMI1_TX0_N-Pad160)
- Module1 pad 163: /CM5_HighSpeed/USB3-1-D_P -> unconnected-(Module1B-USB3-1-D_P-Pad163)
- Module1 pad 164: /CM5_HighSpeed/HDMI1_CK_P -> unconnected-(Module1B-HDMI1_CLK_P-Pad164)
- Module1 pad 165: /CM5_HighSpeed/USB3-1-D_N -> unconnected-(Module1B-USB3-1-D_N-Pad165)
- Module1 pad 166: /CM5_HighSpeed/HDMI1_CK_N -> unconnected-(Module1B-HDMI1_CLK_N-Pad166)
- Module1 pad 169: /CM5_HighSpeed/USB3-1-TX_N -> unconnected-(Module1B-USB3-1-TX_N-Pad169)
- Module1 pad 17: /CM5_GPIO ( Ethernet, GPIO, SDCARD)/ETH_LEDG -> unconnected-(Module1A-Ethernet_nLED2(3.3v)-Pad17)
- Module1 pad 171: /CM5_HighSpeed/USB3-1-TX_P -> unconnected-(Module1B-USB3-1-TX_P-Pad171)
- Module1 pad 35: /CM5_GPIO ( Ethernet, GPIO, SDCARD)/ID_SC -> /CM5_HighSpeed/SCL1
- Module1 pad 36: /CM5_GPIO ( Ethernet, GPIO, SDCARD)/ID_SD -> /CM5_HighSpeed/SDA1
- Module1 pad 78: /CM5_GPIO ( Ethernet, GPIO, SDCARD)/GPIO_VREF -> /+3.3v
- Module1 pad 88: /CM5_GPIO ( Ethernet, GPIO, SDCARD)/+1.8v -> unconnected-(Module1A-+1.8v_(Output)-Pad88)
- Module1 pad 90: /CM5_GPIO ( Ethernet, GPIO, SDCARD)/+1.8v -> unconnected-(Module1A-+1.8v_(Output)-Pad90)
- R2 pad 1: Net-(U3-LEDY_K) -> /LoRa/+3.3v_ESP
- R2 pad 2: /CM5_GPIO ( Ethernet, GPIO, SDCARD)/ETH_LEDG -> /LoRa/ADDR_HIGH
- R3 pad 1: Net-(U3-LEDG_K) -> /LoRa/+5v_USB
- R3 pad 2: /CM5_GPIO ( Ethernet, GPIO, SDCARD)/ETH_LEDY -> GND
- R4 pad 1: /CM5_GPIO ( Ethernet, GPIO, SDCARD)/+1.8v -> /LoRa/+3.3v
- R4 pad 2: /CM5_GPIO ( Ethernet, GPIO, SDCARD)/GPIO_VREF -> /LoRa/ENABLE
- R5 pad 1: /+3.3v -> /LoRa/+3.3v
- R5 pad 2: /CM5_GPIO ( Ethernet, GPIO, SDCARD)/GPIO_VREF -> /LoRa/BOOT_MODE
- R6 pad 1: /CM5_GPIO ( Ethernet, GPIO, SDCARD)/GPIO_VREF -> /+3.3v
- R7 pad 1: /CM5_GPIO ( Ethernet, GPIO, SDCARD)/GPIO_VREF -> /+3.3v
- TP1 pad 1: Net-(D3-K) -> /LoRa/+3.3v_ESP
- U1 pad 1: /CM5_GPIO ( Ethernet, GPIO, SDCARD)/TRD3_P -> /LoRa/VIN
- U1 pad 2: /CM5_GPIO ( Ethernet, GPIO, SDCARD)/TRD3_N -> GND
- U1 pad 3: GND -> /LoRa/+3.3v_ESP
- U2 pad 1: /CM5_GPIO ( Ethernet, GPIO, SDCARD)/TRD1_P -> GND
- U2 pad 10: /CM5_GPIO ( Ethernet, GPIO, SDCARD)/TRD1_P -> unconnected-(U2-IO17-Pad10)
- U2 pad 2: /CM5_GPIO ( Ethernet, GPIO, SDCARD)/TRD1_N -> /LoRa/+3.3v_ESP
- U2 pad 3: GND -> /LoRa/ENABLE
- U2 pad 4: /CM5_GPIO ( Ethernet, GPIO, SDCARD)/TRD0_N -> unconnected-(U2-IO4-Pad4)
- U2 pad 5: /CM5_GPIO ( Ethernet, GPIO, SDCARD)/TRD0_P -> unconnected-(U2-IO5-Pad5)
- U2 pad 6: /CM5_GPIO ( Ethernet, GPIO, SDCARD)/TRD0_P -> unconnected-(U2-IO6-Pad6)
- U2 pad 7: /CM5_GPIO ( Ethernet, GPIO, SDCARD)/TRD0_N -> unconnected-(U2-IO7-Pad7)
- U2 pad 8: GND -> unconnected-(U2-IO15-Pad8)
- U2 pad 9: /CM5_GPIO ( Ethernet, GPIO, SDCARD)/TRD1_N -> unconnected-(U2-IO16-Pad9)
- U3 pad 1: /CM5_GPIO ( Ethernet, GPIO, SDCARD)/TRD0_P -> /LoRa/VIN
- U3 pad 2: /CM5_GPIO ( Ethernet, GPIO, SDCARD)/TRD0_N -> GND
- U3 pad 3: /CM5_GPIO ( Ethernet, GPIO, SDCARD)/TRD1_P -> /LoRa/+3.3v_LoRa
Routing:
- net /+3.3v: track 331.7 -> 10.2 mm, vias 11 -> 0
- net /+5v: track 284.2 -> 119.1 mm, vias 25 -> 10
- net /CM5_GPIO ( Ethernet, GPIO, SDCARD)/VBAT: track 154.8 -> 0.00 mm, vias 2 -> 0
- net /CM5_GPIO ( Ethernet, GPIO, SDCARD)/nPWR_LED: track 130.0 -> 0.00 mm, vias 2 -> 0
- net GND: track 764.8 -> 639.4 mm, vias 476 -> 267
- net Net-(Module1A-LED_nACT): track 114.7 -> 0.00 mm, vias 4 -> 0
- net /CM5_GPIO ( Ethernet, GPIO, SDCARD)/GPIO2: track 122.2 -> 10.5 mm
- net /CM5_HighSpeed/PCIE_TX_N: track 109.5 -> 0.00 mm, vias 2 -> 0
- net /CM5_HighSpeed/PCIE_TX_P: track 109.5 -> 0.00 mm, vias 2 -> 0
- net /CM5_HighSpeed/PCIE_RX_N: track 107.9 -> 0.00 mm, vias 2 -> 0
- net /CM5_HighSpeed/PCIE_RX_P: track 107.8 -> 0.00 mm, vias 2 -> 0
- net /CM5_GPIO ( Ethernet, GPIO, SDCARD)/GPIO3: track 119.5 -> 12.3 mm
- net /CM5_GPIO ( Ethernet, GPIO, SDCARD)/GPIO_VREF: track 103.9 -> 0.00 mm
- net /CM5_HighSpeed/PCIE_CLK_N: track 103.8 -> 0.00 mm, vias 2 -> 0
- net /CM5_HighSpeed/PCIE_CLK_P: track 103.8 -> 0.00 mm, vias 2 -> 0
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- removed copper zone on B.Cu, net /+5v
- removed copper zone on B.Cu, net /CM5_HighSpeed/VBUS
- removed copper zone on F.Cu, net /PCIe-M2/M2_3v3
Other:
- board size 160 x 90 mm -> 59.7 x 85.6 mm
- board text added: "1"
- board text added: "16"
- board text added: "2"
- board text added: "4"
- board text added: "8"
- board text added: "Built-in USB"
- board text added: "EEPROM wr. disable"
- board text added: "ESP32"
- board text added: "ID_SD, ID_SD SEL Arrow for CAM1"
- board text added: "In case of a surge, refill with IMB Magic Smoke"
- board text added: "Remove R6 and R7 for ID_SC and ID_SD if not using CAM/DISP 1"
- board text added: "USB3.0"
- board text added: "eMMC Boot disable"
- board text removed: "Battery CR2032"
- board text removed: "Compute Module 5 IO Board"
- board text removed: "Ethernet"
- board text removed: "FAN"
- board text removed: "Fit for 1.8V GPIO"
- board text removed: "Fit for 3.3V GPIO"
- board text removed: "Fit jumper to disable eMMC Boot"
- board text removed: "Fit jumper to disable writing to EEPROM"
- board text removed: "Fit two jumpers for CAM/DISP 1"
- board text removed: "HDMI1"
- board text removed: "M.2 M Key"
- board text removed: "POE"
- board text removed: "Power Button"
- board text removed: "R2"
- board text removed: "USB3"
