File: CM5IO.kicad_sch (KiCad schematic)
At the start: 12 parts, among them J11 USB_C_Receptacle_USB2.0

Commit message: whatever
Parts:
- removed H1, H2, H3, H4, H5, H6, H7, H8: MountingHole, CM5IO:MountingHole_2.7mm_M2.5_DIN965, symbol Mechanical:MountingHole
- added H10: GND_SOLDERPOINT, Connector_Wire:SolderWirePad_1x01_SMD_5x10mm, symbol Mechanical:MountingHole_Pad_MP
- added H9: VIN_SOLDERPOINT, Connector_Wire:SolderWirePad_1x01_SMD_5x10mm, symbol Mechanical:MountingHole_Pad_MP
- added J1: POWER TERMINAL, TerminalBlock:TerminalBlock_bornier-2_P5.08mm, symbol Connector:Screw_Terminal_01x02
Connections:
- net GND: now also H10.1 (MP), J1.2 (Pin_2)
- new net VIN: H9.1 (MP), J1.1 (Pin_1)
- no-connect marks 2 -> 12
Other:
- removed sheet PCIe-M2
- added sheet PSU (psu.kicad_sch)
- sheet CM5_GPIO ( Ethernet, GPIO, SDCARD) ports: added ID_SC_CAM1, ID_SD_CAM1; removed ID_SC, ID_SD
- note added: "Connectors ------- SDCARD 40way RPI Jumpers Fan"
- note removed: "Connectors ------ M2 MKey"
- note removed: "Connectors ------- Ethernet SDCARD 40way RPI Jumpers Fan Battery"
- moved on the sheet: C18, C9
