File: CM5_GPIO.kicad_sch (KiCad schematic)
At the start: 29 parts, among them J14 JST_SHBM04B-SRSS-TB, J2 Conn_02x07_Odd_Even, J3 Conn_01x03, J7 Micro_SD_Card_Det, J8 THD-20-R, J9 THD-02-R, SW1 Right angle Tact button, U1 TPD4EUSB30, U18 RT9742GGJ5, U2 TPD4EUSB30, U3 MagJack-A70-112-331N126

Commit message: whatever
Parts:
- removed BT1: Battery_Cell, CM5IO:BatteryHolder_Keystone_3034_1x20mm, symbol Device:Battery_Cell
- removed C1: 100n, Capacitor_SMD:C_0402_1005Metric, symbol Device:C
- removed J14: JST_SHBM04B-SRSS-TB, Connector_JST:JST_SH_BM04B-SRSS-TB_1x04-1MP_P1.00mm_Vertical, symbol Connector_Generic:Conn_01x04
- removed J3: Conn_01x03, Connector_PinHeader_2.54mm:PinHeader_1x03_P2.54mm_Vertical, symbol Connector_Generic:Conn_01x03
- removed J9: THD-02-R, Connector_PinHeader_2.54mm:PinHeader_2x02_P2.54mm_Vertical, symbol Connector_Generic:Conn_02x02_Odd_Even
- removed R11: 10K 1%, Resistor_SMD:R_0402_1005Metric, symbol Device:R
- removed R2, R3: 470R, Resistor_SMD:R_0402_1005Metric, symbol Device:R
- removed R4: nf, Resistor_SMD:R_0805_2012Metric_Pad1.20x1.40mm_HandSolder, symbol Device:R
- removed R5: 0R, Resistor_SMD:R_0805_2012Metric_Pad1.20x1.40mm_HandSolder, symbol Device:R
- removed TP2, TP4: TestPoint, TestPoint:TestPoint_Pad_2.0x2.0mm, symbol Connector:TestPoint
- removed U1, U2: TPD4EUSB30, Package_SON:USON-10_2.5x1.0mm_P0.5mm, symbol CM5IO:TPD4EUSB30
- removed U3: MagJack-A70-112-331N126, CM5IO:TRJG0926HENL, symbol CM5IO:MagJack-A70-112-331N126
- added JP8: BT_WIFI_DISABLE, Jumper:SolderJumper-3_P2.0mm_Open_TrianglePad1.0x1.5mm, symbol Jumper:SolderJumper_3_Open
- added TP5: TP +3V3, TestPoint:TestPoint_Pad_2.0x2.0mm, symbol Connector:TestPoint
- J2: value Conn_02x07_Odd_Even -> Conn_02x06_Odd_Even; footprint Connector_PinHeader_2.54mm:PinHeader_2x07_P2.54mm_Vertical -> Connector_PinHeader_2.00mm:PinHeader_2x06_P2.00mm_Vertical; symbol Connector_Generic:Conn_02x07_Odd_Even -> Connector_Generic:Conn_02x06_Odd_Even; Field4 Toby -> (none); Field5 THD-07-R -> (none); Field6 THD-07-R -> (none); Field7 Toby -> (none); Part Description PinHeader_2x07_P2.54mm_Vertical -> PinHeader_2x06_P2.54mm_Vertical
- SW1: footprint Button_Switch_THT:SW_Tactile_SPST_Angled_PTS645Vx58-2LFS -> Button_Switch_SMD:SW_Push_1P1T_NO_CK_KMR2; Field5 PTS645VH58-2LFS -> (none); Field6 PTS645VH58-2LFS -> (none); Field7 CK -> (none); Part Description Right angle through hole Tact switch -> (none)
- TP6: renamed from TP5; value TestPoint -> TP nPWR
- TP7: renamed from TP3; value TestPoint -> TP nACT
Connections:
- net GPIO_VREF is gone; now on net +3.3v: Module1.78 (GPIO_VREF(1.8v/3.3v_Input))
- net +1.8v: no longer Module1.88 (+1.8v_(Output)), Module1.90 (+1.8v_(Output))
- net +3.3v: now also TP5.1
- net BT_nDis: now also JP8.3 (B)
- net GND: now also JP8.2 (C); no longer J2.13 (Pin_13)
- net PMIC_ENABLE: now also J2.10 (Pin_10); no longer J2.12 (Pin_12)
- net PWR_BUT: now also J2.12 (Pin_12); no longer J2.14 (Pin_14)
- net USBOTG: now also J2.8 (Pin_8); no longer J2.10 (Pin_10)
- net WL_nDis: now also JP8.1 (A)
- net ETH_LEDG: no longer names the net of Module1.17 (Ethernet_nLED2(3.3v))
- net ETH_LEDY: no longer names the net of Module1.15 (Ethernet_nLED3(3.3v))
- net ID_SC: no longer names the net of J8.28 (Pin_28)
- net ID_SC: no longer Module1.35 (ID_SC)
- net ID_SD: no longer names the net of J8.27 (Pin_27)
- net ID_SD: no longer Module1.36 (ID_SD)
- new net ID_SC_CAM1: Module1.35 (ID_SC)
- new net ID_SD_CAM1: Module1.36 (ID_SD)
- no-connect marks 9 -> 14
Other:
- note removed: "Ethernet"
- note removed: "Ethernet POE Protection"
- note removed: "FAN connector"
- note removed: "Not Fitted header"
- note removed: "POE Header"
- note removed: "R2 : Pullup added for Fans that don't have a strong internal pullup"
- note removed: "R2 : Simplify nPWR_LED Drive"
- moved on the sheet: C5, D1, J7, R10, R13, TP6, U18
