File: CM5_HighSpeed.kicad_sch (KiCad schematic)
At the start: 19 parts, among them J10 690-019-298-412, J12 USB3_A, J16 Conn_01x22_Female, J22 690-019-298-412, J5 Conn_01x22_Female, J6 THD-02-R, U12 RT9742SNGV, U6 AP22653W6

Commit message: whatever
Parts:
- removed J10: 690-019-298-412, CM5IO:EDAC 690-019-298-412, symbol CM5IO:HDMI_A_1.4
- removed J6: THD-02-R, Connector_PinHeader_2.54mm:PinHeader_2x02_P2.54mm_Vertical, symbol Connector_Generic:Conn_02x02_Odd_Even
- J12: footprint CM5IO:MTCONN_UBAF30-D2011 -> Connector_USB:USB3_A_Molex_48393-001; symbol CM5IO:USB3_A -> Connector:USB3_A; Field5 UBAF30-D2011 -> 48393-0003; Field6 UBAF30-D2011 -> 48393; Field7 Mtconn -> MOLEX; Part Description Dual USB 3 connector -> USB 3.0 A connector
- J22: value 690-019-298-412 -> 46765-1301; footprint CM5IO:EDAC 690-019-298-412 -> CM5IO:CONN_467651301_MOL; symbol CM5IO:HDMI_A_1.4 -> Connector:HDMI_D_1.4; Field5 2614936 -> 2614867; Field6 690-019-298-412 -> 46765-1301; Field7 EDAC -> MOLEX; Field8 UCON00802 -> (none); Part Description HDMI Connector, Right Angle, 19 Contacts, Receptacle, Surfa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 -> 0.40mm Pitch Micro HDMI Connector, Right-Angle Receptacle, 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
Connections:
- net GPIO_VREF is gone; now on net +3.3v: R6.1, R7.1
- net SCL1 is gone; now on net ID_SC: J16.20 (Pin_20), R7.2
- net SDA1 is gone; now on net ID_SD: J16.21 (Pin_21), R6.2
- net GND: now also J12.4 (GND), J12.7 (DRAIN), J22.10 (D0S), J22.13 (CKS), J22.16 (GND), J22.4 (D2S), J22.7 (D1S), J22.SH; no longer J12.A4 (GND), J12.A7 (DRAIN), J12.B4 (GND), J12.B7 (DRAIN), J22.11 (CKS), J22.17 (GND), J22.2 (D2S), J22.5 (D1S), J22.8 (D0S), J22.SH1 (SH), J22.SH2 (SH), J22.SH3 (SH), J22.SH4 (SH)
- net HDMI0_CEC: now also J22.15 (CEC); no longer J22.13 (CEC)
- net HDMI0_CK_N: now also J22.14 (CK-); no longer J22.12 (CK-)
- net HDMI0_CK_P: now also J22.12 (CK+); no longer J22.10 (CK+)
- net HDMI0_D0_N: now also J22.11 (D0-); no longer J22.9 (D0-)
- net HDMI0_D0_P: now also J22.9 (D0+); no longer J22.7 (D0+)
- net HDMI0_D1_N: now also J22.8 (D1-); no longer J22.6 (D1-)
- net HDMI0_D1_P: now also J22.6 (D1+); no longer J22.4 (D1+)
- net HDMI0_D2_N: now also J22.5 (D2-); no longer J22.3 (D2-)
- net HDMI0_D2_P: now also J22.3 (D2+); no longer J22.1 (D2+)
- net HDMI0_HOTPLUG: now also J22.1 (HPD/HEAC-); no longer J22.19 (HPD/HEAC-)
- net HDMI0_SCL: now also J22.17 (SCL); no longer J22.15 (SCL)
- net HDMI0_SDA: now also J22.18 (SDA); no longer J22.16 (SDA)
- net HDMI_5v: now also J22.19 (+5V); no longer J22.18 (+5V)
- net USB3-0-D_N: now also J12.2 (D-); no longer J12.A2 (D-)
- net USB3-0-D_P: now also J12.3 (D+); no longer J12.A3 (D+)
- net USB3-0-RX_N: now also J12.5 (SSRX-); no longer J12.A6 (SSRX+)
- net USB3-0-RX_P: now also J12.6 (SSRX+); no longer J12.A5 (SSRX-)
- net USB3-0-TX_N: now also J12.8 (SSTX-); no longer J12.A9 (SSTX+)
- net USB3-0-TX_P: now also J12.9 (SSTX+); no longer J12.A8 (SSTX-)
- net VBUS: now also J12.1 (VBUS); no longer J12.A1 (VBUS), J12.B1 (VBUS)
- net HDMI1_CEC: no longer names the net of Module1.149 (HDMI1_CEC)
- net HDMI1_CK_N: no longer names the net of Module1.166 (HDMI1_CLK_N)
- net HDMI1_CK_P: no longer names the net of Module1.164 (HDMI1_CLK_P)
- net HDMI1_D0_N: no longer names the net of Module1.160 (HDMI1_TX0_N)
- net HDMI1_D0_P: no longer names the net of Module1.158 (HDMI1_TX0_P)
- net HDMI1_D1_N: no longer names the net of Module1.154 (HDMI1_TX1_N)
- net HDMI1_D1_P: no longer names the net of Module1.152 (HDMI1_TX1_P)
- net HDMI1_D2_N: no longer names the net of Module1.148 (HDMI1_TX2_N)
- net HDMI1_D2_P: no longer names the net of Module1.146 (HDMI1_TX2_P)
- net HDMI1_HOTPLUG: no longer names the net of Module1.143 (HDMI1_HOTPLUG)
- net HDMI1_SCL: no longer names the net of Module1.147 (HDMI1_SCL)
- net HDMI1_SDA: no longer names the net of Module1.145 (HDMI1_SDA)
- net PCIE_CLK_N: no longer names the net of Module1.112 (PCIe_CLK_N)
- net PCIE_CLK_P: no longer names the net of Module1.110 (PCIe_CLK_P)
- net PCIE_PWR_EN: no longer names the net of Module1.106 (PCIE_PWR_EN)
- net PCIE_RX_N: no longer names the net of Module1.118 (PCIe_RX_N)
- net PCIE_RX_P: no longer names the net of Module1.116 (PCIe_RX_P)
- net PCIE_TX_N: no longer names the net of Module1.124 (PCIe_TX_N)
- net PCIE_TX_P: no longer names the net of Module1.122 (PCIe_TX_P)
- net PCIE_nCLKREQ: no longer names the net of Module1.102 (PCIe_nCLKREQ)
- net PCIE_nRST: no longer names the net of Module1.109 (PCIe_nRST)
- net PCIE_nWAKE: no longer names the net of Module1.104 (PCIE_nWAKE)
- net USB3-1-D_N: no longer names the net of Module1.165 (USB3-1-D_N)
- net USB3-1-D_N: no longer J12.B2 (D-)
- net USB3-1-D_P: no longer names the net of Module1.163 (USB3-1-D_P)
- net USB3-1-D_P: no longer J12.B3 (D+)
- net USB3-1-RX_N: no longer names the net of Module1.157 (USB3-1-RX_N)
- net USB3-1-RX_N: no longer J12.B6 (SSRX+)
- net USB3-1-RX_P: no longer names the net of Module1.159 (USB3-1-RX_P)
- net USB3-1-RX_P: no longer J12.B5 (SSRX-)
- net USB3-1-TX_N: no longer names the net of Module1.169 (USB3-1-TX_N)
- net USB3-1-TX_N: no longer J12.B9 (SSTX+)
- net USB3-1-TX_P: no longer names the net of Module1.171 (USB3-1-TX_P)
- net USB3-1-TX_P: no longer J12.B8 (SSTX-)
- no-connect marks 4 -> 31
Other:
- note removed: "Jumpers to be fitted if DPHY1 is used"
- note removed: "Stacked USB connectors"
- moved on the sheet: C12, C13, C2, C3, C7, C8, R12, R6, R7, U12, U6
