File: CM5IO/CM5IO.kicad_pcb (KiCad board)
At the start: 4 copper layers, 59.7 x 78 mm, 62 parts, among them J1 POWER TERMINAL, J11 USB_C_Receptacle_USB2.0, J12 USB3_A, J16 Conn_01x22_Female, J2 Conn_02x06_Odd_Even, J22 46765-1301, J4 J_PSU_EN, J5 Conn_01x22_Female, J7 Micro_SD_Card_Det, J8 THD-20-R, SW1 Right angle Tact button, U12 RT9742SNGV, U18 RT9742GGJ5, U6 AP22653W6

Commit message: post-review fixes
Parts:
- added J14: JST_SHBM04B-SRSS-TB, Connector_JST:JST_SH_BM04B-SRSS-TB_1x04-1MP_P1.00mm_Vertical, B.Cu at (196.6, 103.3)
- added R11: 10K 1%, Resistor_SMD:R_0402_1005Metric, F.Cu at (198.9, 100.7)
Routing:
- net GND: track 775.4 -> 791.0 mm
- net /+5v: track 303.8 -> 317.7 mm, vias 32 -> 34
- net /CM5_GPIO ( Ethernet, GPIO, SDCARD)/TACHO: track 0.00 -> 5.01 mm, vias 0 -> 1
- net /+3.3v: track 197.2 -> 200.1 mm, vias 8 -> 9
- net /CM5_GPIO ( Ethernet, GPIO, SDCARD)/PWM: track 0.00 -> 2.68 mm, vias 0 -> 1
- net /CM5_GPIO ( Ethernet, GPIO, SDCARD)/GPIO25: track 26.3 -> 27.8 mm
- net /CM5_GPIO ( Ethernet, GPIO, SDCARD)/GPIO20: track 43.4 -> 44.7 mm
- net /CM5_GPIO ( Ethernet, GPIO, SDCARD)/GPIO16: track 40.9 -> 42.0 mm
- net /CM5_HighSpeed/USB3-0-TX_P: track 27.7 -> 28.3 mm
- net /CM5_HighSpeed/USB3-0-RX_P: track 29.0 -> 29.6 mm
Other:
- board text added: "0"
- board text added: "0 mm"
- board text added: "0.0152 mm"
- board text added: "0.02"
- board text added: "0.03048 mm"
- board text added: "0.035 mm"
- board text added: "0.0994 mm"
- board text added: "0.1000 mm / 0.1250 mm"
- board text added: "0.2000 mm"
- board text added: "0.7 mm"
- board text added: "1"
- board text added: "1.0602 mm"
- board text added: "3.8"
- board text added: "4"
- board text added: "4.5"
- board text added: "59.6900 mm x 77.9780 mm"
- board text added: "B.Cu"
- board text added: "B.Mask"
- board text added: "B.Paste"
- board text added: "B.Silkscreen"
- board text added: "BOARD CHARACTERISTICS"
- board text added: "Board Thickness:"
- board text added: "Board overall dimensions:"
- board text added: "Bottom Silk Screen"
- board text added: "Bottom Solder Mask"
- board text added: "Bottom Solder Paste"
- board text added: "Castellated pads:"
- board text added: "Color"
- board text added: "Copper Finish:"
- board text added: "Copper Layer Count:"
- board text added: "Dielectric"
- board text added: "Edge card connectors:"
- board text added: "Epsilon R"
- board text added: "F.Cu"
- board text added: "F.Mask"
- board text added: "F.Paste"
- board text added: "F.Silkscreen"
- board text added: "FAN"
- board text added: "FR4"
- board text added: "Green"
- board text added: "Impedance Control:"
- board text added: "In1.Cu"
- board text added: "In2.Cu"
- board text added: "JLC"
- board text added: "Layer Name"
- board text added: "Loss Tangent"
- board text added: "Material"
- board text added: "Min hole diameter:"
- board text added: "Min track/spacing:"
- board text added: "No"
- board text added: "None"
- board text added: "Not specified"
- board text added: "Plated Board Edge:"
- board text added: "Thickness (mm)"
- board text added: "Top Silk Screen"
- board text added: "Top Solder Mask"
- board text added: "Top Solder Paste"
- board text added: "Type"
- board text added: "Yes"
- board text added: "copper"
- board text added: "core"
- board text added: "prepreg"
- board text removed: "Board thickness : 1.6mm Finished copper weight inners : 24.9um or greater Finished copper weight outers : 35um or greater Board finish : OSP Material type : FR4 Colour of solder resists : Green Colour of silk screens : White Only on the top side Board to : UL94-V0 TG >=130 50R trace width 0.13mm@ 3GHz 90R diff pair width 0.147 spacing 0.253mm @ 2.5GHz 100R diff pair width 0.127 spacing 0.253mm @ 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"

Commit message: post-reveiw fixes
Parts:
- C13: moved to B.Cu
- moved C13 4.15 mm to (152.8, 89.2), turned to -90 degrees
Routing:
- net /CM5_GPIO ( Ethernet, GPIO, SDCARD)/CAM_GPIO1: track 49.5 -> 52.5 mm
- net /CM5_HighSpeed/SDA0: track 49.2 -> 52.0 mm
- net GND: track 791.0 -> 788.2 mm, vias 333 -> 304
- net /CM5_GPIO ( Ethernet, GPIO, SDCARD)/CAM_GPIO0: track 53.5 -> 56.1 mm
- net /CM5_HighSpeed/SCL0: track 48.8 -> 51.1 mm
- net /CM5_HighSpeed/DPHY1_D3_P: track 22.6 -> 24.7 mm
- net /CM5_HighSpeed/DPHY1_D3_N: track 22.6 -> 24.7 mm
- net /CM5_HighSpeed/DPHY1_D1_P: track 25.3 -> 27.3 mm
- net /CM5_HighSpeed/DPHY1_D1_N: track 25.3 -> 27.3 mm
- net /CM5_HighSpeed/DPHY1_D0_P: track 26.5 -> 28.3 mm
- net /CM5_HighSpeed/DPHY1_D0_N: track 26.5 -> 28.3 mm
- net /CM5_GPIO ( Ethernet, GPIO, SDCARD)/USBOTG: track 46.1 -> 44.7 mm
- net /CM5_HighSpeed/HDMI0_SDA: track 16.9 -> 18.1 mm
- net /CM5_HighSpeed/DPHY1_D2_P: track 26.5 -> 27.7 mm
- net /CM5_HighSpeed/DPHY1_D2_N: track 26.5 -> 27.7 mm
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
Commit message: post-review fixes
Routing:
- net /CM5_HighSpeed/HDMI0_SCL: track 10.0 -> 20.2 mm
- net GND: vias 304 -> 303

Commit message: final changes before ordering the design
Other:
- board text added: "100R"
- board text added: "90R"
