File: CM5IO/psu.kicad_sch (KiCad schematic)
At the start: 20 parts, among them J4 J_PSU_EN

Commit message: DRC fixes after changing via size. fixed too small cap in PSU.
Parts:
- CP1: footprint Capacitor_Tantalum_SMD:CP_EIA-3528-21_Kemet-B_HandSolder -> Capacitor_Tantalum_SMD:CP_EIA-6032-28_Kemet-C_HandSolder
Changed lines of the file:
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@@
 			)
 		)
-		(property "Footprint" "Capacitor_Tantalum_SMD:CP_EIA-3528-21_Kemet-B_HandSolder"
+		(property "Footprint" "Capacitor_Tantalum_SMD:CP_EIA-6032-28_Kemet-C_HandSolder"
 			(at 101.6 83.82 0)
 			(effects
@@
 			)
 		)
-		(property "Description" "Tantalum, Kemet-B, 10uF@35V min."
+		(property "Description" "Tantalum, Kemet-C, 10uF@35V min."
 			(at 101.6 83.82 0)
 			(effects
