File: CM5IO_top/killswitch.kicad_sch (KiCad schematic)
At the start: 11 parts, among them Q1 AO3401A, Q2 Q_NPN_BEC, Q3 Q_NPN_BEC, Q4 AO3401A, SW3 FORCE_PWR

Commit message: upper board finished (I hope)
Parts:
- added R16: 10K, Resistor_SMD:R_0805_2012Metric_Pad1.20x1.40mm_HandSolder, symbol Device:R_Small
Connections:
- net GND: now also R16.2
- net PSU_EN_CTL: now also R16.1
Other:
- note added: "Solder pulldown to disable automatic startup of PSU"
Changed lines of the file:
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@@
 	(generator_version "9.0")
 	(paper "A4")
+	(text "Solder pulldown to \ndisable automatic \nstartup of PSU"
+		(exclude_from_sim no)
+		(at 119.888 133.35 0)
+		(effects
+			(font
+				(size 1.27 1.27)
+			)
+			(justify left)
+		)
+	)
 	(junction
 		(at 95.25 125.73)
@@
 	)
 	(junction
+		(at 115.57 115.57)
+		(diameter 0)
+		(color 0 0 0 0)
+	)
+	(junction
 		(at 95.25 67.31)
 		(diameter 0)
@@
 	(wire
 		(pts
+			(xy 115.57 115.57) (xy 123.19 115.57)
+		)
+		(stroke
+			(width 0)
+			(type default)
+		)
+	)
+	(wire
+		(pts
+			(xy 115.57 135.89) (xy 115.57 151.13)
+		)
+		(stroke
+			(width 0)
+			(type default)
+		)
+	)
+	(wire
+		(pts
 			(xy 77.47 80.01) (xy 80.01 80.01)
 		)
@@
 	(wire
 		(pts
-			(xy 109.22 115.57) (xy 113.03 115.57)
+			(xy 109.22 115.57) (xy 115.57 115.57)
 		)
 		(stroke
@@
 	(wire
 		(pts
+			(xy 115.57 151.13) (xy 95.25 151.13)
+		)
+		(stroke
+			(width 0)
+			(type default)
+		)
+	)
+	(wire
+		(pts
 			(xy 86.36 88.9) (xy 86.36 92.71)
 		)
@@
 		(pts
 			(xy 95.25 151.13) (xy 95.25 153.67)
+		)
+		(stroke
+			(width 0)
+			(type default)
+		)
+	)
+	(wire
+		(pts
+			(xy 115.57 115.57) (xy 115.57 130.81)
 		)
 		(stroke
@@
 	(hierarchical_label "PSU_EN_CTL"
 		(shape output)
-		(at 113.03 115.57 0)
+		(at 123.19 115.57 0)
 		(effects
 			(font
@@
 					(unit 1)
 				)
+			)
+		)
+	)
+	(symbol
+		(lib_id "Device:R_Small")
+		(at 115.57 133.35 0)
+		(unit 1)
+		(exclude_from_sim no)
+		(in_bom yes)
+		(on_board yes)
+		(dnp no)
+		(property "Reference" "R16"
+			(at 117.856 132.588 0)
+			(effects
+				(font
+					(size 1.016 1.016)
+				)
+			)
+		)
+		(property "Value" "10K"
+			(at 117.856 134.112 0)
+			(effects
+				(font
+					(size 1.27 1.27)
+				)
+			)
+		)
+		(property "Footprint" "Resistor_SMD:R_0805_2012Metric_Pad1.20x1.40mm_HandSolder"
+			(at 115.57 133.35 0)
+			(effects
+				(font
+					(size 1.27 1.27)
+				)
+				(hide yes)
+			)
+		)
+		(property "Datasheet" "~"
+			(at 115.57 133.35 0)
+			(effects
+				(font
+					(size 1.27 1.27)
+				)
+				(hide yes)
+			)
+		)
+		(property "Description" "Resistor, small symbol"
+			(at 115.57 133.35 0)
+			(effects
+				(font
+					(size 1.27 1.27)
+				)
+				(hide yes)
+			)
+		)
+		(pin "1"
+		)
+		(pin "2"
+		)
+		(instances
+			(project "CM5IO_top"
+				(path "/45032d28-0209-4e67-a308-47ee4cd3805e/73c647b5-bc1b-4f18-9452-dba8bbf7e1d4"
+					(reference "R16")
+					(unit 1)
+				)
